Commit message: Update LegBot model parameters: mass, collision box, COM
- base mass: 6.583964 -> 7.09 kg
- thigh mass: 1.55038 -> 1.456 kg (x4)
- foot mass: 0.04 -> 0.025 kg (x4)
- base collision box: 27x21x11 cm
- base COM: (-1.2, 0.2, 0.1) cm
- synced to vbot_mujoco

Files: 7 XML/URDF files + changelog

File: legbot_description/urdf/legbot_description.urdf (robot description, URDF)
Before this commit: robot legbot_description, 17 links, 16 joints
Links:
- link FL_foot: mass 0.04 -> 0.025
- link FL_thigh: mass 1.55038 -> 1.456
- link FR_foot: mass 0.04 -> 0.025
- link FR_thigh: mass 1.55038 -> 1.456
- link RL_foot: mass 0.04 -> 0.025
- link RL_thigh: mass 1.55038 -> 1.456
- link RR_foot: mass 0.04 -> 0.025
- link RR_thigh: mass 1.55038 -> 1.456
- link base: mass 6.583964 -> 7.09; geometry collision box size=0.27 0.21 0.11; visual mesh filename=package://legbot_description/meshes/base_link.STL

File: resources/legbot/urdf/legbot.urdf (robot description, URDF)
Before this commit: robot legbot_description, 17 links, 16 joints
Links:
- link FL_foot: mass 0.04 -> 0.025
- link FL_thigh: mass 1.55038 -> 1.456
- link FR_foot: mass 0.04 -> 0.025
- link FR_thigh: mass 1.55038 -> 1.456
- link RL_foot: mass 0.04 -> 0.025
- link RL_thigh: mass 1.55038 -> 1.456
- link RR_foot: mass 0.04 -> 0.025
- link RR_thigh: mass 1.55038 -> 1.456
- link base: mass 6.583964 -> 7.09; geometry collision box size=0.169204 0.157994 0.083746; collision box size=0.27 0.21 0.11

Commit message: Update LegBot project files and training artifacts

File: legbot_description/urdf/legbot_description.urdf (robot description, URDF)
Before this commit: robot legbot_description, 17 links, 16 joints
Joints:
- joint FL_hip_joint: origin xyz=0.18453 0.051 0 rpy=0 0 0 -> xyz=0.18453 0.051 0.012 rpy=0 0 0
- joint FR_hip_joint: origin xyz=0.18453 -0.051 0 rpy=0 0 0 -> xyz=0.18453 -0.051 0.012 rpy=0 0 0
- joint RL_hip_joint: origin xyz=-0.18453 0.051 0 rpy=0 0 0 -> xyz=-0.18453 0.051 0.012 rpy=0 0 0
- joint RR_hip_joint: origin xyz=-0.18453 -0.051 0 rpy=0 0 0 -> xyz=-0.18453 -0.051 0.012 rpy=0 0 0
